File: CapBankBreakout/CapBankBreakout.kicad_pcb (KiCad board)
At the start: 2 copper layers, 382 x 90 mm, 36 parts

Commit message: commit 2
hi brady
Parts:
- added J1: 7461097, ALF70C103EH400:7461097, F.Cu at (496.6, 109.2)
- added J2: 7461097, ALF70C103EH400:7461097, F.Cu at (496.6, 146.1)
- added REF**: Symbol_Danger_CopperTop_Small, Symbol:Symbol_Danger_CopperTop_Small, F.Cu at (93.6, 168.0)
- C1, C10, C11, C12, C13, C14, C2, C3, C31, C32, C4, C5, C6, C7, C8, C9: moved to F.Cu
- moved C9 617.1 mm to (134.8, 97.4), turned to 0 degrees
- moved C10 543.4 mm to (156.8, 158.1)
- moved C11 491.6 mm to (178.8, 97.4), turned to 0 degrees
- moved C12 415.6 mm to (200.8, 158.1)
- moved C13 368.5 mm to (222.8, 97.4), turned to 0 degrees
- moved REF** 365.9 mm to (495.9, 127.0), turned to 90 degrees
- moved REF** 365.9 mm to (495.9, 127.0), turned to -90 degrees
- moved C8 355.8 mm to (464.8, 158.1), turned to 180 degrees
- moved C7 321.0 mm to (442.8, 97.5), turned to 0 degrees
- moved REF** 313.7 mm to (104.7, 128.6), turned to -90 degrees
- moved REF** 313.7 mm to (104.7, 128.6), turned to 90 degrees
- moved C14 289.0 mm to (244.8, 158.1)
- moved C6 259.9 mm to (398.8, 97.5), turned to 0 degrees
- moved C31 251.1 mm to (266.8, 97.4), turned to 0 degrees
- moved C5 217.9 mm to (354.8, 97.5), turned to 0 degrees
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Other:
- board size 382 x 90 mm -> 421.8 x 120.1 mm
- board text added: "Capacitor Bank Breakout R1 {dblquote}Kinetic Antenna{dblquote} Senior Design Missouri S&T 2024"
