File: CapBankBreakout/CapBankBreakout.kicad_pcb (KiCad board)
At the start: 2 copper layers, 421.8 x 120.1 mm, 39 parts, among them J1 7461097, J2 7461097

Commit message: redesign 1
mouse bites inserted.
Parts:
- removed J1, J2: 7461097, ALF70C103EH400:7461097
- removed the REF** at (495.9, 127.0) (x2)
- added J**: CAP_SIDE_1, ALF70C103EH400:CAP_SIDE_1, F.Cu at (105.0, 104.8)
- added REF**: HV-warning, ALF70C103EH400:HV-warning, B.Cu at (496.8, 245.0)
- added REF**: HV-warning, ALF70C103EH400:HV-warning, F.Cu at (135.5, 214.2)
- added REF**: HV-warning, ALF70C103EH400:HV-warning, F.Cu at (506.8, 150.0)
- added REF**: HV-warning, ALF70C103EH400:HV-warning, F.Cu at (506.8, 245.0)
- added REF**: Symbol_Danger_CopperTop_Small, Symbol:Symbol_Danger_CopperTop_Small, F.Cu at (110.0, 285.0)
- added REF**: CAP_SIDE_2, ALF70C103EH400:CAP_SIDE_2, F.Cu at (105.0, 200.0)
- added REF**: HV-warning, ALF70C103EH400:HV-warning, B.Cu at (135.5, 214.2)
- added REF**: HV-warning, ALF70C103EH400:HV-warning, B.Cu at (496.8, 150.0)
- added V1: BATT_PWR_VIA, ALF70C103EH400:via, F.Cu at (496.3, 130.9)
- added V2: BATT_PWR_VIA, ALF70C103EH400:via, F.Cu at (135.6, 169.0)
- added V3: BATT_PWR_VIA, ALF70C103EH400:via, F.Cu at (496.2, 264.0)
- added V4: BATT_PWR_VIA, ALF70C103EH400:via, F.Cu at (135.5, 225.9)
- added mouse-bite-5mm-slot: VAL**, Panelization:mouse-bite-5mm-slot, F.Cu at (350.0, 197.5)
- added mouse-bite-5mm-slot (x2): VAL**, Panelization:mouse-bite-5mm-slot, F.Cu at (137.5, 197.5)
- added mouse-bite-5mm-slot: VAL**, Panelization:mouse-bite-5mm-slot, F.Cu at (292.5, 197.5)
- added mouse-bite-5mm-slot: VAL**, Panelization:mouse-bite-5mm-slot, F.Cu at (505.0, 197.5)
- moved C29 225.8 mm to (326.9, 275.5)
- moved C17 225.8 mm to (194.9, 275.5)
- moved C19 225.8 mm to (238.9, 275.5)
- moved C21 225.8 mm to (282.9, 275.5)
- moved C23 225.8 mm to (370.9, 275.5)
- moved C24 225.8 mm to (414.9, 275.5)
- moved C27 225.8 mm to (458.9, 275.5)
- moved C15 225.7 mm to (151.1, 275.5)
- moved C16 225.4 mm to (173.1, 214.6)
- moved C18 225.4 mm to (217.1, 214.6)
- moved C20 225.4 mm to (261.1, 214.6)
- moved C22 225.4 mm to (349.1, 214.6)
- moved C25 225.4 mm to (393.1, 214.6)
- moved C26 225.4 mm to (437.1, 214.6)
- moved C28 225.4 mm to (481.1, 214.6)
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Connections:
- net PCB1_CAP+ renamed VBUS
- net PCB1_CAP- renamed GNDPWR
Other:
- board size 421.8 x 120.1 mm -> 422 x 185 mm
- board text added: "CAPACITOR?? I HARDLY KNOW HER!!!"
- board text added: "Capacitor Bank Breakout R1 {dblquote}Kinetic Antenna{dblquote} Senior Design 23-24 Missouri S&T ECE Department"
- board text added: "MJR, 2024"
- board text removed: "Capacitor Bank Breakout R1 {dblquote}Kinetic Antenna{dblquote} Senior Design Missouri S&T 2024"

Commit message: board review changes made
rounded corners, cosmetic changes
Other:
- outline, holes or cut-outs redrawn
- board text added: "CAPACITOR? I HARDLY KNOW HER!"
- board text removed: "CAPACITOR?? I HARDLY KNOW HER!!!"
Changed lines of the file:
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@@
   (gr_circle (center 120 275.19) (end 120 272.904)
     (stroke (width 0.1) (type default)) (fill none) (layer "Edge.Cuts"))
-  (gr_line (start 527 195) (end 527 105)
+  (gr_line (start 527 190) (end 527 110)
     (stroke (width 0.1) (type default)) (layer "Edge.Cuts"))
-  (gr_line (start 105 200) (end 137.5 200)
+  (gr_line (start 110 200) (end 137.5 200)
     (stroke (width 0.1) (type default)) (layer "Edge.Cuts"))
   (gr_line (start 340 200) (end 302.5 200)
     (stroke (width 0.1) (type default)) (layer "Edge.Cuts"))
+  (gr_arc (start 110 195) (mid 106.464466 193.535534) (end 105 190)
+    (stroke (width 0.1) (type default)) (layer "Edge.Cuts"))
   (gr_arc (start 505 200) (mid 502.5 197.5) (end 505 195)
+    (stroke (width 0.1) (type default)) (layer "Edge.Cuts"))
+  (gr_arc (start 105 110) (mid 106.464466 106.464466) (end 110 105)
     (stroke (width 0.1) (type default)) (layer "Edge.Cuts"))
   (gr_line (start 350 195) (end 495 195)
@@
   (gr_circle (center 120 180) (end 120 177.714)
     (stroke (width 0.1) (type default)) (fill none) (layer "Edge.Cuts"))
-  (gr_line (start 527 200) (end 527 290)
+  (gr_line (start 527 205) (end 527 285)
     (stroke (width 0.1) (type default)) (layer "Edge.Cuts"))
   (gr_arc (start 340 195) (mid 342.5 197.5) (end 340 200)
@@
   (gr_arc (start 292.5 195) (mid 295 197.5) (end 292.5 200)
     (stroke (width 0.1) (type default)) (layer "Edge.Cuts"))
-  (gr_line (start 527 290) (end 105 290)
+  (gr_line (start 522 290) (end 110 290)
     (stroke (width 0.1) (type default)) (layer "Edge.Cuts"))
-  (gr_line (start 505 200) (end 527 200)
+  (gr_arc (start 110 290) (mid 106.464466 288.535534) (end 105 285)
+    (stroke (width 0.1) (type default)) (layer "Edge.Cuts"))
+  (gr_arc (start 522 200) (mid 525.535524 201.464476) (end 527 205)
+    (stroke (width 0.1) (type default)) (layer "Edge.Cuts"))
+  (gr_line (start 505 200) (end 522 200)
     (stroke (width 0.1) (type default)) (layer "Edge.Cuts"))
   (gr_circle (center 120 119.83) (end 120 117.544)
@@
   (gr_arc (start 302.5 200) (mid 300 197.5) (end 302.5 195)
     (stroke (width 0.1) (type default)) (layer "Edge.Cuts"))
-  (gr_line (start 105 290) (end 105 200)
+  (gr_line (start 105 285) (end 105 205)
     (stroke (width 0.1) (type default)) (layer "Edge.Cuts"))
   (gr_line (start 495 200) (end 350 200)
@@
   (gr_arc (start 137.5 195) (mid 140 197.5) (end 137.5 200)
     (stroke (width 0.1) (type default)) (layer "Edge.Cuts"))
-  (gr_line (start 527 105) (end 105 105)
+  (gr_line (start 522 105) (end 110 105)
     (stroke (width 0.1) (type default)) (layer "Edge.Cuts"))
-  (gr_line (start 105 105) (end 105 195)
+  (gr_line (start 105 110) (end 105 190)
+    (stroke (width 0.1) (type default)) (layer "Edge.Cuts"))
+  (gr_arc (start 527 285) (mid 525.535548 288.535568) (end 522 290)
+    (stroke (width 0.1) (type default)) (layer "Edge.Cuts"))
+  (gr_arc (start 522 105) (mid 525.535534 106.464466) (end 527 110)
     (stroke (width 0.1) (type default)) (layer "Edge.Cuts"))
   (gr_line (start 302.5 195) (end 340 195)
     (stroke (width 0.1) (type default)) (layer "Edge.Cuts"))
-  (gr_line (start 505 195) (end 527 195)
+  (gr_line (start 505 195) (end 522 195)
     (stroke (width 0.1) (type default)) (layer "Edge.Cuts"))
   (gr_line (start 292.5 200) (end 147.5 200)
     (stroke (width 0.1) (type default)) (layer "Edge.Cuts"))
-  (gr_line (start 137.5 195) (end 105 195)
+  (gr_arc (start 527 190) (mid 525.535534 193.535534) (end 522 195)
     (stroke (width 0.1) (type default)) (layer "Edge.Cuts"))
-  (gr_text "CAPACITOR?? \nI HARDLY KNOW HER!!!" (at 522.5 245 90) (layer "B.SilkS")
+  (gr_line (start 137.5 195) (end 110 195)
+    (stroke (width 0.1) (type default)) (layer "Edge.Cuts"))
+  (gr_arc (start 105 205) (mid 106.464466 201.464466) (end 110 200)
+    (stroke (width 0.1) (type default)) (layer "Edge.Cuts"))
+  (gr_text "CAPACITOR?\nI HARDLY KNOW HER!" (at 522.5 245 90) (layer "B.SilkS")
     (effects (font (size 4 4) (thickness 1) bold) (justify bottom mirror))
   )
-  (gr_text "CAPACITOR?? \nI HARDLY KNOW HER!!!" (at 522.5 150 90) (layer "B.SilkS")
+  (gr_text "CAPACITOR?\nI HARDLY KNOW HER!" (at 522.5 150 90) (layer "B.SilkS")
     (effects (font (size 4 4) (thickness 1) bold) (justify bottom mirror))
   )
@@
     (effects (font (size 2 2) (thickness 0.5) bold))
   )
-  (gr_text "MJR, 2024" (at 517 194) (layer "F.SilkS")
+  (gr_text "MJR, 2024" (at 515 194) (layer "F.SilkS")
     (effects (font (size 1 1) (thickness 0.15)) (justify left bottom))
   )
-  (gr_text "MJR, 2024" (at 517 289) (layer "F.SilkS")
+  (gr_text "MJR, 2024" (at 515 289) (layer "F.SilkS")
     (effects (font (size 1 1) (thickness 0.15)) (justify left bottom))
   )
@@
     (pts (xy 527 104.83) (xy 527 194.935118))
     (height -5.5)
-    (gr_text "90.1051 mm" (at 531.35 149.882559 90) (layer "User.2")
+    (gr_text "3547.4456 mils" (at 531.35 149.882559 90) (layer "User.2")
       (effects (font (size 1 1) (thickness 0.15)))
     )
@@
     (pts (xy 527 104.83) (xy 105 104.83))
     (height -202.67)
-    (gr_text "422.0000 mm" (at 316 306.35) (layer "User.2")
+    (gr_text "16614.1732 mils" (at 316 306.35) (layer "User.2")
       (effects (font (size 1 1) (thickness 0.15)))
     )
