File: CapBankBreakout/CapBankBreakout.kicad_pcb (KiCad board)
At the start: 2 copper layers, 422 x 185 mm, 53 parts

Commit message: holes added and double board generated
Parts:
- added G***: LOGO, MRDT_Silkscreens:z_sig_MaxRyan_25x6.6mm, F.Cu at (504.6, 191.4)
- added G***: LOGO, MRDT_Silkscreens:z_sig_MaxRyan_25x6.6mm, F.Cu at (504.6, 286.8)
Other:
- outline, holes or cut-outs redrawn
- board text added: "Capacitor Bank Breakout R1 Kinetic Antenna Senior Design 23-24 Missouri S&T ECE Department"
- board text added: "REF**"
- board text added: "V+"
- board text added: "V-"
- board text removed: "Capacitor Bank Breakout R1 {dblquote}Kinetic Antenna{dblquote} Senior Design 23-24 Missouri S&T ECE Department"
